Commit message: usd converter 4.5.0

File: source/extensions/orbit.surgical.assets/data/Robots/MOPS/mopsV2.urdf (robot description, URDF)
Before this commit: robot mops, 21 links, 20 joints
Links:
- link tool_jaw1: mass None -> 0.01
- link tool_jaw2: mass None -> 0.01
Joints:
- joint tool_pitch: limit lower=-1.3962634015954636 upper=1.3962634015954636 effort=0.25 velocity=6.283185307179586 -> lower=-1.3962634015954636 upper=1.3962634015954636 effort=50 velocity=6.283185307179586
- joint tool_roll: limit lower=-4.537856055185257 upper=4.537856055185257 effort=0.3 velocity=6.283185307179586 -> lower=-4.537856055185257 upper=4.537856055185257 effort=30 velocity=6.283185307179586
