Commit message: FIX urdf

File: source/extensions/orbit.surgical.assets/data/Robots/MOPS/mops.urdf (robot description, URDF)
Before this commit: robot mops, 18 links, 17 joints
Links:
- removed link lnd_main_insertion_link_3
- added link lnd_rod_link, mass 0.000001; collision mesh filename=meshes/lnd_main_insertion_link_3_collisions.obj scale=1. 1. 1.; visual mesh filename=meshes/lnd_main_insertion_link_3_visuals.obj scale=1. 1. 1.
- link kuka_link_0: geometry visual mesh filename=meshes/kuka_link_0_visuals.obj scale=1. 1. 1.
- link kuka_link_1: geometry collision cylinder length=0.208 radius=0.07; collision sphere radius=0.07
- link kuka_link_2: geometry collision cylinder length=0.208 radius=0.07; collision sphere radius=0.07
- link kuka_link_3: geometry collision cylinder length=0.208 radius=0.07; collision sphere radius=0.07
- link kuka_link_4: geometry collision cylinder length=0.208 radius=0.07; collision sphere radius=0.07
- link kuka_link_5: geometry collision cylinder length=0.198 radius=0.07; collision sphere radius=0.07
- link kuka_link_6: geometry collision sphere radius=0.08; visual mesh filename=meshes/kuka_link_6_visuals.obj scale=1. 1. 1.
- link kuka_link_7: geometry collision cylinder length=0.05 radius=0.04; visual mesh filename=meshes/kuka_link_7_visuals.obj scale=1. 1. 1.
- link lnd_tool_gripper1_link: geometry collision mesh filename=meshes/lnd_tool_gripper1_link_collisions.obj scale=1. 1. 1.; visual mesh filename=meshes/lnd_tool_gripper1_link_visuals.obj scale=1. 1. 1.
- link lnd_tool_gripper2_link: geometry collision mesh filename=meshes/lnd_tool_gripper2_link_collisions.obj scale=1. 1. 1.; visual mesh filename=meshes/lnd_tool_gripper2_link_visuals.obj scale=1. 1. 1.
- link lnd_tool_pitch_link: geometry collision mesh filename=meshes/lnd_tool_pitch_link_collisions_mesh_0.obj scale=1. 1. 1.; collision mesh filename=meshes/lnd_tool_pitch_link_collisions_mesh_1.obj scale=1. 1. 1.
- link lnd_tool_roll_link: geometry collision mesh filename=meshes/lnd_tool_roll_link_collisions_mesh_0.obj scale=1. 1. 1.; collision mesh filename=meshes/lnd_tool_roll_link_collisions_mesh_1.obj scale=1. 1. 1.
- link lnd_tool_yaw_link: geometry collision mesh filename=meshes/lnd_tool_yaw_link_collisions_mesh_0.obj scale=1. 1. 1.; collision mesh filename=meshes/lnd_tool_yaw_link_collisions_mesh_1.obj scale=1. 1. 1.
Joints:
- removed joint lnd_main_insertion_joint_3
- removed joint root_joint
- added joint kuka_lwr_root_joint: type fixed, parent kuka_lwr, child kuka_link_0, origin xyz=0. 0. 0. rpy=0. 0. 0.
- added joint lnd_rod_joint: type fixed, parent lnd_base_link, child lnd_rod_link, origin xyz=0. 0. -0.61421  rpy=0. 0. 1.5707963
- joint Xi_housing_joint: origin xyz=-0.015 0. 0.06 rpy=0. 1.5707964 0. -> xyz=-0.015 -0. 0.0600001 rpy=-0. 1.5707964 0. ; parent lnd_main_insertion_link_3 -> lnd_rod_link
- joint kuka_joint_2: axis 0. -1. 0. -> 0. 1. 0.; limit lower=-2.0943948 upper=2.0943948 effort=5000. velocity=1.9198619 -> lower=-2.0943946 upper=2.0943946 effort=5000. velocity=1.9198619; origin xyz=0 0 0.2005 rpy=0 0 0 -> xyz=0. 0. 0.2005 rpy=3.1415927 0. 0. 
- joint kuka_joint_3: axis 0 0 1 -> 0. 0. 1.; limit lower=-2.96706 upper=2.96706 effort=5000. velocity=2.234021 -> lower=-2.96706 upper=2.96706 effort=5000. velocity=2.2340209; origin xyz=0 0 0.2 rpy=0 0 0 -> xyz=0. 0. -0.2 rpy=3.1415927 0. 0. 
- joint kuka_joint_4: axis 0 1 0 -> 0. 1. 0.; limit lower=-2.0943948 upper=2.0943948 effort=5000. velocity=2.234021 -> lower=-2.0943946 upper=2.0943946 effort=5000. velocity=2.2340209; origin xyz=0 0 0.2 rpy=0 0 0 -> xyz=0. 0. 0.2 rpy=0. 0. 0.
- joint kuka_joint_5: axis 0 0 1 -> 0. 0. 1.; limit lower=-2.96706 upper=2.96706 effort=5000. velocity=3.56047 -> lower=-2.96706 upper=2.96706 effort=5000. velocity=3.5604701; origin xyz=0 0 0.20 rpy=0 0 0 -> xyz=0. 0. 0.2 rpy=0. 0. 0.
- joint kuka_joint_6: axis 0 -1 0 -> 0. 1. 0.; limit lower=-2.0943948 upper=2.0943948 effort=5000. velocity=3.211405 -> lower=-2.0943946 upper=2.0943946 effort=5000. velocity=3.211405; origin xyz=0 0 0.19 rpy=0 0 0 -> xyz=0. 0. 0.19 rpy=3.1415927 0. 0. 
- joint kuka_joint_7: axis 0 0 1 -> 0. 0. 1.; origin xyz=0 0 0.078 rpy=0 0 0 -> xyz=0. 0. -0.078 rpy=3.1415927 0. 0. 
- joint lnd_root_joint: origin xyz=0.614720316841551 0.088064119102809 0.001429763596620 rpy=0. 1.570796326795 0. -> xyz=0. 0.612 0.132 rpy=1.570796326795 0. 3.14159265359 
- joint lnd_tool_gripper1_joint: origin xyz=0. 0. 0. rpy=0. 0. 0. -> xyz=-0. 0. 0. rpy=0.0000001 0.0000001 -0.0000002
- joint lnd_tool_gripper2_joint: origin xyz=0. 0. 0. rpy=0. 0. 0. -> xyz=-0. 0. 0. rpy=0.0000001 0.0000001 -0.0000002
- joint lnd_tool_pitch_joint: origin xyz=0. 0. 0. rpy=-1.5707964 0. 1.5707964 -> xyz=-0.0000001 -0. 0.  rpy=-1.5707965 0. 1.5707963
- joint lnd_tool_roll_joint: limit lower=-4.5378997 upper=4.5378997 effort=6000. velocity=2.0999999 -> lower=-4.5378992 upper=4.5378992 effort=6000. velocity=2.0999999; origin xyz=0. 0. 0.59862  rpy=0.-1.5707963 -1.5707963 -> xyz=0. -0. 0.5986201 rpy=-1.5707963 -1.5707963 0. ; parent lnd_main_insertion_link_3 -> lnd_rod_link
- joint lnd_tool_tip_joint: origin xyz=0. 0.0093 0.  rpy=-1.5707964 0. 0.  -> xyz=0. 0.0093 0.  rpy=-1.5707963 0.0000001 -0.0000002
- joint lnd_tool_yaw_joint: origin xyz=0. 0. -0.0091 rpy=-1.5707964 0. 1.5707964 -> xyz=0. 0. -0.0091 rpy=-1.5707964 -0.0000001 1.5707964

Commit message: changed to kuka iwwa14

File: source/extensions/orbit.surgical.assets/data/Robots/MOPS/mops.urdf (robot description, URDF)
Before this commit: robot mops, 18 links, 17 joints
Links:
- removed link Xi_housing_link
- removed link kuka_lwr
- removed link lnd_base_link
- removed link lnd_rod_link
- removed link lnd_tool_gripper1_link
- removed link lnd_tool_gripper2_link
- removed link lnd_tool_pitch_link
- removed link lnd_tool_roll_link
- removed link lnd_tool_tip_link
- removed link lnd_tool_yaw_link
- added link kuka_link_ee
- added link tool_base
- added link tool_housing; visual box size=0.06 0.045 0.08
- added link tool_jaw0
- added link tool_jaw1; collision mesh filename=meshes/lnd_tip/lnd_tool_gripper1_link_collisions_xform_coll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 scale=0.00009 0.0004 0.0001; visual mesh filename=meshes/lnd_tip/jaw.stl
- added link tool_jaw2; collision mesh filename=meshes/lnd_tip/lnd_tool_gripper2_link_collisions_xform_coll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 scale=0.00009 0.0004 0.0001; visual mesh filename=meshes/lnd_tip/jaw.stl
- added link tool_jaw_hinge
- added link tool_rotation; collision mesh filename=meshes/lnd_tip/roll.stl scale=1.01 1.01 1.01; visual mesh filename=meshes/lnd_tip/roll.stl
- added link tool_shaft; collision cylinder length=0.5365 radius=0.004; visual cylinder length=0.5365 radius=0.004
- added link tool_tcp0
- added link tool_tcp1
- added link tool_tcp2
- added link tool_wrist; collision mesh filename=meshes/lnd_tip/wrist.stl scale=1.01 1.01 1.01; visual mesh filename=meshes/lnd_tip/wrist.stl
- link kuka_link_0: mass 2. -> 7.050378; geometry collision mesh filename=meshes/iiwa14/collision/link_0.stl; visual mesh filename=meshes/iiwa14/visual/link_0.dae
- link kuka_link_1: mass 2. -> 5.289529; geometry collision mesh filename=meshes/iiwa14/collision/link_1.stl; visual mesh filename=meshes/iiwa14/visual/link_1.dae
- link kuka_link_2: mass 2. -> 5.688888; geometry collision mesh filename=meshes/iiwa14/collision/link_2.stl; visual mesh filename=meshes/iiwa14/visual/link_2.dae
- link kuka_link_3: mass 2. -> 3.461245; geometry collision mesh filename=meshes/iiwa14/collision/link_3.stl; visual mesh filename=meshes/iiwa14/visual/link_3.dae
- link kuka_link_4: mass 2. -> 4.122995; geometry collision mesh filename=meshes/iiwa14/collision/link_4.stl; visual mesh filename=meshes/iiwa14/visual/link_4.dae
- link kuka_link_5: mass 2. -> 1.563756; geometry collision mesh filename=meshes/iiwa14/collision/link_5.stl; visual mesh filename=meshes/iiwa14/visual/link_5.dae
- link kuka_link_6: mass 0.2 -> 2.457878; geometry collision mesh filename=meshes/iiwa14/collision/link_6.stl; visual mesh filename=meshes/iiwa14/visual/link_6.dae
- link kuka_link_7: mass 0.2 -> 0.265331; geometry collision mesh filename=meshes/iiwa14/collision/link_7.stl; visual mesh filename=meshes/iiwa14/visual/link_7.dae
Joints:
- removed joint Xi_housing_joint
- removed joint kuka_joint_1
- removed joint kuka_joint_2
- removed joint kuka_joint_3
- removed joint kuka_joint_4
- removed joint kuka_joint_5
- removed joint kuka_joint_6
- removed joint kuka_joint_7
- removed joint kuka_lwr_root_joint
- removed joint lnd_rod_joint
- removed joint lnd_root_joint
- removed joint lnd_tool_gripper1_joint
- removed joint lnd_tool_gripper2_joint
- removed joint lnd_tool_pitch_joint
- removed joint lnd_tool_roll_joint
- removed joint lnd_tool_tip_joint
- removed joint lnd_tool_yaw_joint
- added joint kuka_A1: type revolute, parent kuka_link_0, child kuka_link_1, origin xyz=0.0 0.0 0.1475 rpy=0 0 0, axis 0.0 0.0 1.0, limit lower=-2.9670597283903604 upper=2.9670597283903604 effort=200 velocity=1.4835298641951802
- added joint kuka_A2: type revolute, parent kuka_link_1, child kuka_link_2, origin xyz=0.0 -0.01 0.2125 rpy=0 0 0, axis 0.0 1.0 0.0, limit lower=-2.0943951023931953 upper=2.0943951023931953 effort=200 velocity=1.4835298641951802
- added joint kuka_A3: type revolute, parent kuka_link_2, child kuka_link_3, origin xyz=0.0 0.01 0.228 rpy=0 0 0, axis 0.0 0.0 1.0, limit lower=-2.9670597283903604 upper=2.9670597283903604 effort=200 velocity=1.7453292519943295
- added joint kuka_A4: type revolute, parent kuka_link_3, child kuka_link_4, origin xyz=0.0 0.0105 0.192 rpy=0 0 0, axis 0.0 -1.0 0.0, limit lower=-2.0943951023931953 upper=2.0943951023931953 effort=200 velocity=1.3089969389957472
- added joint kuka_A5: type revolute, parent kuka_link_4, child kuka_link_5, origin xyz=0.0 -0.0105 0.2075 rpy=0 0 0, axis 0.0 0.0 1.0, limit lower=-2.9670597283903604 upper=2.9670597283903604 effort=200 velocity=2.2689280275926285
- added joint kuka_A6: type revolute, parent kuka_link_5, child kuka_link_6, origin xyz=0.0 -0.0707 0.1925 rpy=0 0 0, axis 0.0 1.0 0.0, limit lower=-2.0943951023931953 upper=2.0943951023931953 effort=200 velocity=2.356194490192345
- added joint kuka_A7: type revolute, parent kuka_link_6, child kuka_link_7, origin xyz=0.0 0.0707 0.091 rpy=0 0 0, axis 0.0 0.0 1.0, limit lower=-3.0543261909900763 upper=3.0543261909900763 effort=200 velocity=2.356194490192345
- added joint kuka_joint_ee: type fixed, parent kuka_link_7, child kuka_link_ee, origin xyz=0 0 0.035 rpy=0 0 0
- added joint tool_base_fixed: type fixed, parent kuka_link_ee, child tool_base, origin xyz=0.05 0 0.174 rpy=0 0 0
- added joint tool_housing_fixed: type fixed, parent tool_base, child tool_housing, origin xyz=-0.03 0 -0.02 rpy=0 0 0
- added joint tool_jaw_hinge_fixed: type fixed, parent tool_wrist, child tool_jaw_hinge, origin xyz=0.0091 0 0 rpy=1.5707963267948966 0 0
- added joint tool_pitch: type revolute, parent tool_rotation, child tool_wrist, origin xyz=0 0 0 rpy=-1.5707963267948966 -1.5707963267948966 0, axis 0 0 1, limit lower=-1.3962634015954636 upper=1.3962634015954636 effort=0.25 velocity=6.283185307179586
- added joint tool_roll: type revolute, parent tool_base, child tool_rotation, origin xyz=0.5455 0 0 rpy=-3.141592653589793 -1.5707963267948966 0, axis 0 0 1, limit lower=-4.537856055185257 upper=4.537856055185257 effort=0.3 velocity=6.283185307179586
- added joint tool_shaft_fixed: type fixed, parent tool_rotation, child tool_shaft, origin xyz=0 0 -0.27725 rpy=0 0 0
- added joint tool_tcp0_fixed: type fixed, parent tool_jaw0, child tool_tcp0, origin xyz=0.009 0 0 rpy=0 0 0
- added joint tool_tcp1_fixed: type fixed, parent tool_jaw1, child tool_tcp1, origin xyz=0.009 0 0 rpy=0 0 0
- added joint tool_tcp2_fixed: type fixed, parent tool_jaw2, child tool_tcp2, origin xyz=0.009 0 0 rpy=0 0 0
- added joint tool_yaw0: type revolute, parent tool_jaw_hinge, child tool_jaw0, origin xyz=0 0 0 rpy=0 0 0, axis 0 0 1, limit lower=-1.3089969389957472 upper=1.3089969389957472 effort=0.2 velocity=6.283185307179586
- added joint tool_yaw1: type revolute, parent tool_jaw_hinge, child tool_jaw1, origin xyz=0 0 0 rpy=0 0 0, axis 0 0 1, limit lower=-1.3089969389957472 upper=1.3089969389957472 effort=0.2 velocity=6.283185307179586
- added joint tool_yaw2: type revolute, parent tool_jaw_hinge, child tool_jaw2, origin xyz=0 0 0 rpy=3.141592653589793 0 0, axis 0 0 1, limit lower=-1.3089969389957472 upper=1.3089969389957472 effort=0.2 velocity=6.283185307179586

Commit message: converted urdf to usd in 5.0.0

File: source/extensions/orbit.surgical.assets/data/Robots/MOPS/mops.urdf (robot description, URDF)
Before this commit: robot mops, 21 links, 20 joints
Joints:
- joint tool_pitch: limit lower=-1.3962634015954636 upper=1.3962634015954636 effort=0.25 velocity=6.283185307179586 -> lower=-1.3962634015954636 upper=1.3962634015954636 effort=50 velocity=6.283185307179586
- joint tool_roll: limit lower=-4.537856055185257 upper=4.537856055185257 effort=0.3 velocity=6.283185307179586 -> lower=-4.537856055185257 upper=4.537856055185257 effort=50 velocity=6.283185307179586

Commit message: usd in 5.0.0

File: source/extensions/orbit.surgical.assets/data/Robots/MOPS/mops.urdf (robot description, URDF)
Before this commit: robot mops, 21 links, 20 joints
Joints:
- joint tool_pitch: limit lower=-1.3962634015954636 upper=1.3962634015954636 effort=0.25 velocity=6.283185307179586 -> lower=-1.3962634015954636 upper=1.3962634015954636 effort=50 velocity=6.283185307179586
- joint tool_roll: limit lower=-4.537856055185257 upper=4.537856055185257 effort=0.3 velocity=6.283185307179586 -> lower=-4.537856055185257 upper=4.537856055185257 effort=30 velocity=6.283185307179586
