Commit message: added weight to tool

File: source/extensions/orbit.surgical.assets/data/Robots/iiwa14/iiwa14.urdf (robot description, URDF)
Before this commit: robot mops, 21 links, 20 joints
Links:
- removed link tool_base
- removed link tool_housing
- removed link tool_jaw0
- removed link tool_jaw1
- removed link tool_jaw2
- removed link tool_jaw_hinge
- removed link tool_rotation
- removed link tool_shaft
- removed link tool_tcp0
- removed link tool_tcp1
- removed link tool_tcp2
- removed link tool_wrist
Joints:
- removed joint tool_base_fixed
- removed joint tool_housing_fixed
- removed joint tool_jaw_hinge_fixed
- removed joint tool_pitch
- removed joint tool_roll
- removed joint tool_shaft_fixed
- removed joint tool_tcp0_fixed
- removed joint tool_tcp1_fixed
- removed joint tool_tcp2_fixed
- removed joint tool_yaw0
- removed joint tool_yaw1
- removed joint tool_yaw2
